File: electrical/sparkfun-pi-hat/pi-hat-v.02-sparkfun.brd (EAGLE design)
At the start: 86.4 x 53.3 mm, 13 parts, among them J1 PIN20X2

Commit message: plate through holes, upload BOM
Parts:
- added H1, H2, H3, H4: MOUNT-PAD-ROUND3.3, holes:3,3-PAD
Other:
- board size 86.4 x 53.3 mm -> 92.7 x 53.3 mm
Changed lines of the file:
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@@
 <layer number="43" name="vRestrict" color="2" fill="10" visible="yes" active="yes"/>
 <layer number="44" name="Drills" color="7" fill="1" visible="no" active="yes"/>
-<layer number="45" name="Holes" color="7" fill="1" visible="no" active="yes"/>
+<layer number="45" name="Holes" color="7" fill="1" visible="yes" active="yes"/>
 <layer number="46" name="Milling" color="3" fill="1" visible="no" active="yes"/>
 <layer number="47" name="Measures" color="7" fill="1" visible="no" active="yes"/>
@@
 <board>
 <plain>
-<wire x1="10.16" y1="6.35" x2="96.52" y2="6.35" width="0.1524" layer="20"/>
+<wire x1="3.81" y1="6.35" x2="96.52" y2="6.35" width="0.1524" layer="20"/>
 <wire x1="96.52" y1="6.35" x2="96.52" y2="59.69" width="0.1524" layer="20"/>
-<wire x1="96.52" y1="59.69" x2="10.16" y2="59.69" width="0.1524" layer="20"/>
-<wire x1="10.16" y1="59.69" x2="10.16" y2="6.35" width="0.1524" layer="20"/>
+<wire x1="96.52" y1="59.69" x2="3.81" y2="59.69" width="0.1524" layer="20"/>
+<wire x1="3.81" y1="59.69" x2="3.81" y2="6.35" width="0.1524" layer="20"/>
 <text x="12.7" y="44.45" size="1.4224" layer="21" rot="R90" align="center">VDD</text>
 <text x="36.83" y="44.45" size="1.4224" layer="21" rot="R90" align="center">VDD</text>
@@
 <text x="57.15" y="7.62" size="1.27" layer="21" align="center">Left Rear</text>
 <text x="77.47" y="7.62" size="1.27" layer="21" align="center">Right Rear</text>
-<text x="50.8" y="34.29" size="1.27" layer="21" align="center">Open Race Scale</text>
-<text x="50.8" y="31.75" size="0.8128" layer="21" align="center">RoaddogLabs PiHat v0.02
+<text x="74.93" y="31.75" size="1.27" layer="21" align="center">Open Race Scale</text>
+<text x="74.93" y="29.21" size="0.8128" layer="21" align="center">RoaddogLabs PiHat v0.02
 https://github.com/RoaddogLabs/open-race-scale
 forked from https://github.com/jenkinsracing/open-race-scale</text>
@@
 </class>
 </classes>
-<designrules name="default">
+<designrules name="SeeedStudio_2layer_DRU_no_angle_20140221">
 <description language="de">&lt;b&gt;EAGLE Design Rules&lt;/b&gt;
 &lt;p&gt;
@@
 necessary adjustments and save your customized
 design rules under a new name.</description>
+<description language="zh">&lt;b&gt;Seeed Studio EAGLE Design Rules&lt;/b&gt;
+</description>
 <param name="layerSetup" value="(1*16)"/>
-<param name="mtCopper" value="0.035mm 0.035mm 0.035mm 0.035mm 0.035mm 0.035mm 0.035mm 0.035mm 0.035mm 0.035mm 0.035mm 0.035mm 0.035mm 0.035mm 0.035mm 0.035mm"/>
-<param name="mtIsolate" value="1.5mm 0.15mm 0.2mm 0.15mm 0.2mm 0.15mm 0.2mm 0.15mm 0.2mm 0.15mm 0.2mm 0.15mm 0.2mm 0.15mm 0.2mm"/>
+<param name="mtCopper" value="0.035mm 0.0175mm 0.035mm 0.035mm 0.035mm 0.035mm 0.035mm 0.035mm 0.035mm 0.035mm 0.035mm 0.035mm 0.035mm 0.035mm 0.0175mm 0.035mm"/>
+<param name="mtIsolate" value="1.5mm 1.1mm 0.2mm 0.15mm 0.2mm 0.15mm 0.2mm 0.15mm 0.2mm 0.15mm 0.2mm 0.15mm 0.2mm 0.15mm 0.2mm"/>
 <param name="mdWireWire" value="6mil"/>
 <param name="mdWirePad" value="6mil"/>
@@
 <param name="mdPadVia" value="6mil"/>
 <param name="mdViaVia" value="6mil"/>
-<param name="mdSmdPad" value="6mil"/>
-<param name="mdSmdVia" value="6mil"/>
-<param name="mdSmdSmd" value="6mil"/>
-<param name="mdViaViaSameLayer" value="6mil"/>
+<param name="mdSmdPad" value="0mil"/>
+<param name="mdSmdVia" value="0mil"/>
+<param name="mdSmdSmd" value="0mil"/>
+<param name="mdViaViaSameLayer" value="8mil"/>
 <param name="mnLayersViaInSmd" value="2"/>
-<param name="mdCopperDimension" value="40mil"/>
-<param name="mdDrill" value="6mil"/>
+<param name="mdCopperDimension" value="10mil"/>
+<param name="mdDrill" value="10mil"/>
 <param name="mdSmdStop" value="0mil"/>
 <param name="msWidth" value="6mil"/>
-<param name="msDrill" value="0.35mm"/>
-<param name="msMicroVia" value="9.99mm"/>
+<param name="msDrill" value="12mil"/>
+<param name="msMicroVia" value="12mil"/>
 <param name="msBlindViaRatio" value="0.5"/>
 <param name="rvPadTop" value="0.25"/>
@@
 <param name="rlMinPadBottom" value="10mil"/>
 <param name="rlMaxPadBottom" value="20mil"/>
-<param name="rlMinViaOuter" value="8mil"/>
+<param name="rlMinViaOuter" value="6mil"/>
 <param name="rlMaxViaOuter" value="20mil"/>
-<param name="rlMinViaInner" value="8mil"/>
+<param name="rlMinViaInner" value="6mil"/>
 <param name="rlMaxViaInner" value="20mil"/>
 <param name="rlMinMicroViaOuter" value="4mil"/>
@@
 <param name="psTop" value="-1"/>
 <param name="psBottom" value="-1"/>
-<param name="psFirst" value="-1"/>
+<param name="psFirst" value="0"/>
 <param name="psElongationLong" value="100"/>
 <param name="psElongationOffset" value="100"/>
 <param name="mvStopFrame" value="1"/>
 <param name="mvCreamFrame" value="0"/>
-<param name="mlMinStopFrame" value="4mil"/>
-<param name="mlMaxStopFrame" value="4mil"/>
+<param name="mlMinStopFrame" value="2mil"/>
+<param name="mlMaxStopFrame" value="2mil"/>
 <param name="mlMinCreamFrame" value="0mil"/>
 <param name="mlMaxCreamFrame" value="0mil"/>
-<param name="mlViaStopLimit" value="0mil"/>
+<param name="mlViaStopLimit" value="100mil"/>
 <param name="srRoundness" value="0"/>
 <param name="srMinRoundness" value="0mil"/>
@@
 <param name="checkAngle" value="0"/>
 <param name="checkFont" value="1"/>
-<param name="checkRestrict" value="1"/>
+<param name="checkRestrict" value="0"/>
 <param name="useDiameter" value="13"/>
 <param name="maxErrors" value="50"/>
@@
 <element name="J8" library="SparkFun-Connectors" package="1X05" value="" x="60.96" y="20.32"/>
 <element name="J9" library="SparkFun-Connectors" package="1X05" value="" x="83.82" y="20.32"/>
+<element name="H1" library="holes" package="3,3-PAD" value="MOUNT-PAD-ROUND3.3" x="8.89" y="54.61"/>
+<element name="H2" library="holes" package="3,3-PAD" value="MOUNT-PAD-ROUND3.3" x="91.44" y="54.61"/>
+<element name="H3" library="holes" package="3,3-PAD" value="MOUNT-PAD-ROUND3.3" x="8.89" y="11.43"/>
+<element name="H4" library="holes" package="3,3-PAD" value="MOUNT-PAD-ROUND3.3" x="91.44" y="11.43"/>
 </elements>
 <signals>
